File: POWERBOARD v3/power_v3.0/5.3to5V.kicad_sch (KiCad schematic)
At the start: 7 parts, among them IC2 MAX25301AATB_V+T

Commit message: updated file names and added hierarchy schematic, problem with ERC bc of GND
Parts:
- renumbered 5V to 5V1, 5V to 5V2, C6 to C10, C10 to C6, IC2 to IC1
Connections:
- net output_at_5.3 is gone; now on net input_at_5.3: C10.1, IC1.1 (IN_1), IC1.2 (IN_2), IC1.4 (EN)
- net output_at_5: now also IC1.7 (OUTS)
- net input_at_5.3: now reaches IC1.5 (SELA)
- net input_at_5.3: now also IC1.6 (SELB)
Changed lines of the file:
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@@
 		)
 	)
-	(text_box "texte pas up to date\nLDO: MAX25301A\nVIN: 5V3 (1.7V-5.5V)\nVOUT: 5V (SELA=GND, SELB=NC)\nImax: 1A (Ilim 1.4A typ)\nDropout: 100mV max @ 1A\nCIN/COUT: 10uF / 10uF (4uF min after derating)\nCBYP: 10nF OUT-to-BYP (soft-start 5V/ms)\nOUTS: Kelvin back to load"
+	(text_box "texte pas up to date\nLDO: MAX25301A\nVIN: 5V3 (1.7V-5.5V)\nVOUT: 5V (SELA=IN, SELB=IN)\nImax: 1A (Ilim 1.4A typ)\nDropout: 100mV max @ 1A\nCIN/COUT: 10uF / 10uF (4uF min after derating)\nCBYP: 10nF OUT-to-BYP (soft-start 5V/ms)\nOUTS: Kelvin back to load"
 		(exclude_from_sim no)
 		(at 118.11 124.4747 0)
@@
 	)
 	(junction
+		(at 175.26 71.12)
+		(diameter 0)
+		(color 0 0 0 0)
+	)
+	(junction
 		(at 170.18 71.12)
 		(diameter 0)
@@
 		(color 0 0 0 0)
 	)
+	(junction
+		(at 128.27 71.12)
+		(diameter 0)
+		(color 0 0 0 0)
+	)
 	(wire
 		(pts
@@
 	(wire
 		(pts
-			(xy 118.11 78.74) (xy 132.08 78.74)
+			(xy 118.11 78.74) (xy 128.27 78.74)
 		)
 		(stroke
@@
 	(wire
 		(pts
-			(xy 118.11 76.2) (xy 132.08 76.2)
+			(xy 118.11 76.2) (xy 121.92 76.2)
 		)
 		(stroke
@@
 	(wire
 		(pts
-			(xy 118.11 81.28) (xy 132.08 81.28)
+			(xy 118.11 81.28) (xy 121.92 81.28)
 		)
 		(stroke
@@
 	(wire
 		(pts
+			(xy 128.27 78.74) (xy 128.27 71.12)
+		)
+		(stroke
+			(width 0)
+			(type default)
+		)
+	)
+	(wire
+		(pts
 			(xy 231.14 64.77) (xy 231.14 76.2)
 		)
@@
 	(wire
 		(pts
-			(xy 73.66 71.12) (xy 85.09 71.12)
+			(xy 175.26 68.58) (xy 175.26 71.12)
+		)
+		(stroke
+			(width 0)
+			(type default)
+		)
+	)
+	(wire
+		(pts
+			(xy 67.31 71.12) (xy 85.09 71.12)
 		)
 		(stroke
@@
 	)
 	(label "output_at_5"
-		(at 175.26 71.12 0)
+		(at 175.26 68.58 0)
 		(effects
 			(font
@@
 	)
 	(label "BYP"
-		(at 129.54 76.2 0)
+		(at 121.92 76.2 0)
 		(effects
 			(font
@@
 		)
 	)
-	(global_label "output_at_5.3"
-		(shape input)
-		(at 73.66 71.12 180)
-		(fields_autoplaced yes)
+	(label "IN"
+		(at 80.01 81.28 0)
 		(effects
 			(font
 				(size 1.27 1.27)
 			)
+			(justify left bottom)
+		)
+	)
+	(label "IN"
+		(at 121.92 81.28 0)
+		(effects
+			(font
+				(size 1.27 1.27)
+			)
+			(justify left bottom)
+		)
+	)
+	(hierarchical_label "input_at_5.3"
+		(shape input)
+		(at 67.31 71.12 180)
+		(effects
+			(font
+				(size 1.27 1.27)
+			)
 			(justify right)
-		)
-		(property "Intersheetrefs" "${INTERSHEET_REFS}"
-			(at 57.7937 71.12 0)
-			(hide yes)
-			(show_name no)
-			(do_not_autoplace no)
-			(effects
-				(font
-					(size 1.27 1.27)
-				)
-				(justify right)
-			)
 		)
 	)
@@
 		(dnp no)
 		(fields_autoplaced yes)
-		(property "Reference" "C6"
+		(property "Reference" "C10"
 			(at 219.71 78.7399 0)
 			(show_name no)
@@
 		(instances
 			(project "power_v3.0"
-				(path "/432bcdcf-747a-4fa0-b87b-096f44260199/866bbf8f-ce37-4fcc-b504-1859f0ec9ca1"
-					(reference "C6")
+				(path "/432bcdcf-747a-4fa0-b87b-096f44260199/d34c4d5c-3529-4589-bd14-5dc8f8f897de"
+					(reference "C10")
 					(unit 1)
 				)
@@
 		(dnp no)
 		(fields_autoplaced yes)
-		(property "Reference" "C10"
+		(property "Reference" "C6"
 			(at 162.56 82.5499 0)
 			(show_name no)
@@
 		(instances
 			(project "power_v3.0"
-				(path "/432bcdcf-747a-4fa0-b87b-096f44260199/866bbf8f-ce37-4fcc-b504-1859f0ec9ca1"
-					(reference "C10")
+				(path "/432bcdcf-747a-4fa0-b87b-096f44260199/d34c4d5c-3529-4589-bd14-5dc8f8f897de"
+					(reference "C6")
 					(unit 1)
 				)
@@
 		(dnp no)
 		(fields_autoplaced yes)
-		(property "Reference" "IC2"
+		(property "Reference" "IC1"
 			(at 102.87 63.5 0)
 			(show_name no)
@@
 		(instances
 			(project "power_v3.0"
-				(path "/432bcdcf-747a-4fa0-b87b-096f44260199/866bbf8f-ce37-4fcc-b504-1859f0ec9ca1"
-					(reference "IC2")
+				(path "/432bcdcf-747a-4fa0-b87b-096f44260199/d34c4d5c-3529-4589-bd14-5dc8f8f897de"
+					(reference "IC1")
 					(unit 1)
 				)
@@
 		(instances
 			(project "power_v3.0"
-				(path "/432bcdcf-747a-4fa0-b87b-096f44260199/866bbf8f-ce37-4fcc-b504-1859f0ec9ca1"
+				(path "/432bcdcf-747a-4fa0-b87b-096f44260199/d34c4d5c-3529-4589-bd14-5dc8f8f897de"
 					(reference "#PWR018")
 					(unit 1)
@@
 		(instances
 			(project "power_v3.0"
-				(path "/432bcdcf-747a-4fa0-b87b-096f44260199/866bbf8f-ce37-4fcc-b504-1859f0ec9ca1"
+				(path "/432bcdcf-747a-4fa0-b87b-096f44260199/d34c4d5c-3529-4589-bd14-5dc8f8f897de"
 					(reference "C11")
 					(unit 1)
@@
 		(instances
 			(project "power_v3.0"
-				(path "/432bcdcf-747a-4fa0-b87b-096f44260199/866bbf8f-ce37-4fcc-b504-1859f0ec9ca1"
+				(path "/432bcdcf-747a-4fa0-b87b-096f44260199/d34c4d5c-3529-4589-bd14-5dc8f8f897de"
 					(reference "#PWR017")
 					(unit 1)
@@
 		(instances
 			(project "power_v3.0"
-				(path "/432bcdcf-747a-4fa0-b87b-096f44260199/866bbf8f-ce37-4fcc-b504-1859f0ec9ca1"
+				(path "/432bcdcf-747a-4fa0-b87b-096f44260199/d34c4d5c-3529-4589-bd14-5dc8f8f897de"
 					(reference "#PWR014")
 					(unit 1)
@@
 		(dnp no)
 		(fields_autoplaced yes)
-		(property "Reference" "5V"
+		(property "Reference" "5V2"
 			(at 186.69 77.4699 0)
 			(show_name no)
@@
 		(instances
 			(project "power_v3.0"
-				(path "/432bcdcf-747a-4fa0-b87b-096f44260199/866bbf8f-ce37-4fcc-b504-1859f0ec9ca1"
-					(reference "5V")
+				(path "/432bcdcf-747a-4fa0-b87b-096f44260199/d34c4d5c-3529-4589-bd14-5dc8f8f897de"
+					(reference "5V2")
 					(unit 1)
 				)
@@
 		(in_pos_files yes)
 		(dnp no)
-		(property "Reference" "5V"
+		(property "Reference" "5V1"
 			(at 170.434 55.118 0)
 			(show_name no)
@@
 		(instances
 			(project "power_v3.0"
-				(path "/432bcdcf-747a-4fa0-b87b-096f44260199/866bbf8f-ce37-4fcc-b504-1859f0ec9ca1"
-					(reference "5V")
+				(path "/432bcdcf-747a-4fa0-b87b-096f44260199/d34c4d5c-3529-4589-bd14-5dc8f8f897de"
+					(reference "5V1")
 					(unit 1)
 				)
@@
 		(instances
 			(project "power_v3.0"
-				(path "/432bcdcf-747a-4fa0-b87b-096f44260199/866bbf8f-ce37-4fcc-b504-1859f0ec9ca1"
+				(path "/432bcdcf-747a-4fa0-b87b-096f44260199/d34c4d5c-3529-4589-bd14-5dc8f8f897de"
 					(reference "D1")
 					(unit 1)

Commit message: Fixed diode layout, added C to VBUS and protection to BUCK-LDO interface
Parts:
- added D4: SOD323, Diode_THT:D_DO-41_SOD81_P10.16mm_Horizontal, symbol Device:D_Zener
- D1: value D_TVS -> PTVS6V0P1UP-QX
Connections:
- net GND: now also D1.2 (A), D4.2 (A); no longer D1.1 (K)
- net input_at_5.3: now also D4.1 (K)
- net output_at_5: now also D1.1 (K); no longer D1.2 (A)
Other:
- moved on the sheet: D1
Changed lines of the file:
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@@
 		(fill
 			(type color)
-			(color 0 0 255 0.1490196078)
+			(color 92 0 255 0.168627451)
 		)
 		(effects
@@
 				(size 1.27 1.27)
 				(thickness 0.1588)
+			)
+			(justify left top)
+		)
+	)
+	(text_box "Clamping value of D3 : 6.0V\n"
+		(exclude_from_sim no)
+		(at 121.92 107.95 0)
+		(size 26.67 6.35)
+		(margins 0.9525 0.9525 0.9525 0.9525)
+		(stroke
+			(width 0)
+			(type solid)
+		)
+		(fill
+			(type none)
+		)
+		(effects
+			(font
+				(size 1.27 1.27)
+			)
+			(justify left top)
+		)
+	)
+	(text_box "Clamping value of D4 : 5.49V\n"
+		(exclude_from_sim no)
+		(at 21.59 80.01 0)
+		(size 26.67 6.35)
+		(margins 0.9525 0.9525 0.9525 0.9525)
+		(stroke
+			(width 0)
+			(type solid)
+		)
+		(fill
+			(type none)
+		)
+		(effects
+			(font
+				(size 1.27 1.27)
 			)
 			(justify left top)
@@
 	)
 	(junction
+		(at 133.35 96.52)
+		(diameter 0)
+		(color 0 0 0 0)
+	)
+	(junction
+		(at 133.35 71.12)
+		(diameter 0)
+		(color 0 0 0 0)
+	)
+	(junction
 		(at 175.26 71.12)
 		(diameter 0)
@@
 	)
 	(junction
-		(at 143.51 96.52)
+		(at 54.61 71.12)
 		(diameter 0)
 		(color 0 0 0 0)
@@
 	)
 	(junction
-		(at 143.51 71.12)
-		(diameter 0)
-		(color 0 0 0 0)
-	)
-	(junction
 		(at 128.27 71.12)
 		(diameter 0)
@@
 	(wire
 		(pts
-			(xy 143.51 80.01) (xy 143.51 71.12)
-		)
-		(stroke
-			(width 0)
-			(type default)
-		)
-	)
-	(wire
-		(pts
 			(xy 80.01 81.28) (xy 87.63 81.28)
 		)
@@
 	(wire
 		(pts
-			(xy 143.51 87.63) (xy 143.51 96.52)
-		)
-		(stroke
-			(width 0)
-			(type default)
-		)
-	)
-	(wire
-		(pts
 			(xy 80.01 78.74) (xy 87.63 78.74)
 		)
@@
 	(wire
 		(pts
-			(xy 121.92 71.12) (xy 143.51 71.12)
+			(xy 121.92 71.12) (xy 158.75 71.12)
 		)
 		(stroke
@@
 	(wire
 		(pts
+			(xy 54.61 86.36) (xy 54.61 96.52)
+		)
+		(stroke
+			(width 0)
+			(type default)
+		)
+	)
+	(wire
+		(pts
 			(xy 179.07 80.01) (xy 175.26 80.01)
 		)
@@
 	(wire
 		(pts
-			(xy 158.75 96.52) (xy 143.51 96.52)
+			(xy 133.35 87.63) (xy 133.35 96.52)
+		)
+		(stroke
+			(width 0)
+			(type default)
+		)
+	)
+	(wire
+		(pts
+			(xy 54.61 96.52) (xy 102.87 96.52)
 		)
 		(stroke
@@
 	(wire
 		(pts
+			(xy 133.35 71.12) (xy 133.35 80.01)
+		)
+		(stroke
+			(width 0)
+			(type default)
+		)
+	)
+	(wire
+		(pts
 			(xy 121.92 73.66) (xy 121.92 71.12)
 		)
@@
 	(wire
 		(pts
-			(xy 143.51 71.12) (xy 158.75 71.12)
-		)
-		(stroke
-			(width 0)
-			(type default)
-		)
-	)
-	(wire
-		(pts
 			(xy 175.26 68.58) (xy 175.26 71.12)
 		)
@@
 	(wire
 		(pts
-			(xy 67.31 71.12) (xy 85.09 71.12)
+			(xy 45.72 71.12) (xy 54.61 71.12)
+		)
+		(stroke
+			(width 0)
+			(type default)
+		)
+	)
+	(wire
+		(pts
+			(xy 54.61 71.12) (xy 54.61 78.74)
+		)
+		(stroke
+			(width 0)
+			(type default)
+		)
+	)
+	(wire
+		(pts
+			(xy 54.61 71.12) (xy 85.09 71.12)
 		)
 		(stroke
@@
 	(wire
 		(pts
-			(xy 143.51 96.52) (xy 102.87 96.52)
+			(xy 102.87 96.52) (xy 158.75 96.52)
 		)
 		(stroke
@@
 	(hierarchical_label "input_at_5.3"
 		(shape input)
-		(at 67.31 71.12 180)
+		(at 45.72 71.12 180)
 		(effects
 			(font
@@
 	)
 	(symbol
+		(lib_id "Device:D_Zener")
+		(at 54.61 82.55 270)
+		(unit 1)
+		(body_style 1)
+		(exclude_from_sim no)
+		(in_bom yes)
+		(on_board yes)
+		(in_pos_files yes)
+		(dnp no)
+		(fields_autoplaced yes)
+		(property "Reference" "D4"
+			(at 57.15 81.2799 90)
+			(show_name no)
+			(do_not_autoplace no)
+			(effects
+				(font
+					(size 1.27 1.27)
+				)
+				(justify left)
+			)
+		)
+		(property "Value" "SOD323"
+			(at 57.15 83.8199 90)
+			(show_name no)
+			(do_not_autoplace no)
+			(effects
+				(font
+					(size 1.27 1.27)
+				)
+				(justify left)
+			)
+		)
+		(property "Footprint" "Diode_THT:D_DO-41_SOD81_P10.16mm_Horizontal"
+			(at 54.61 82.55 0)
+			(hide yes)
+			(show_name no)
+			(do_not_autoplace no)
+			(effects
+				(font
+					(size 1.27 1.27)
+				)
+			)
+		)
+		(property "Datasheet" "https://www.vishay.com/docs/86475/gdz.pdf"
+			(at 54.61 82.55 0)
+			(hide yes)
+			(show_name no)
+			(do_not_autoplace no)
+			(effects
+				(font
+					(size 1.27 1.27)
+				)
+			)
+		)
+		(property "Description" "Zener diode"
+			(at 54.61 82.55 0)
+			(hide yes)
+			(show_name no)
+			(do_not_autoplace no)
+			(effects
+				(font
+					(size 1.27 1.27)
+				)
+			)
+		)
+		(pin "1"
+		)
+		(pin "2"
+		)
+		(instances
+			(project "power_v3.0"
+				(path "/432bcdcf-747a-4fa0-b87b-096f44260199/d34c4d5c-3529-4589-bd14-5dc8f8f897de"
+					(reference "D4")
+					(unit 1)
+				)
+			)
+		)
+	)
+	(symbol
 		(lib_id "N_pulse:MAX25301AATB_V+T")
 		(at 87.63 71.12 0)
@@
 		(instances
 			(project "power_v3.0"
+				(path "/432bcdcf-747a-4fa0-b87b-096f44260199/b63164f7-da09-43bf-9854-ef6b4b4934c1"
+					(reference "IC1")
+					(unit 1)
+				)
 				(path "/432bcdcf-747a-4fa0-b87b-096f44260199/d34c4d5c-3529-4589-bd14-5dc8f8f897de"
 					(reference "IC1")
@@
 	(symbol
 		(lib_id "Device:D_Zener")
-		(at 143.51 83.82 90)
+		(at 133.35 83.82 270)
 		(unit 1)
 		(body_style 1)
@@
 		(fields_autoplaced yes)
 		(property "Reference" "D1"
-			(at 146.05 82.5499 90)
-			(show_name no)
-			(do_not_autoplace no)
-			(effects
-				(font
-					(size 1.27 1.27)
-				)
-				(justify right)
-			)
-		)
-		(property "Value" "D_TVS"
-			(at 146.05 85.0899 90)
-			(show_name no)
-			(do_not_autoplace no)
-			(effects
-				(font
-					(size 1.27 1.27)
-				)
-				(justify right)
+			(at 135.89 82.5499 90)
+			(show_name no)
+			(do_not_autoplace no)
+			(effects
+				(font
+					(size 1.27 1.27)
+				)
+				(justify left)
+			)
+		)
+		(property "Value" "PTVS6V0P1UP-QX"
+			(at 135.89 85.0899 90)
+			(show_name no)
+			(do_not_autoplace no)
+			(effects
+				(font
+					(size 1.27 1.27)
+				)
+				(justify left)
 			)
 		)
 		(property "Footprint" "Diode_THT:D_DO-41_SOD81_P10.16mm_Horizontal"
-			(at 143.51 83.82 0)
-			(hide yes)
-			(show_name no)
-			(do_not_autoplace no)
-			(effects
-				(font
-					(size 1.27 1.27)
-				)
-			)
-		)
-		(property "Datasheet" ""
-			(at 143.51 83.82 0)
+			(at 133.35 83.82 0)
+			(hide yes)
+			(show_name no)
+			(do_not_autoplace no)
+			(effects
+				(font
+					(size 1.27 1.27)
+				)
+			)
+		)
+		(property "Datasheet" "https://assets.nexperia.com/documents/data-sheet/PTVSXP1UP-Q_SER.pdf"
+			(at 133.35 83.82 0)
 			(hide yes)
 			(show_name no)
@@
 		)
 		(property "Description" "Zener diode"
-			(at 143.51 83.82 0)
-			(hide yes)
-			(show_name no)
+			(at 133.35 83.82 0)
+			(hide yes)
+			(show_name no)
