File: POWERBOARD v3/power_v3.0/Conversion battery-5.3V.kicad_sch (KiCad schematic)
At the start: 14 parts, among them U7 TPS62160DSG

Commit message: updated file names and added hierarchy schematic, problem with ERC bc of GND
Parts:
- renumbered Cin3 to Cin1, Cout3 to Cout1, L5 to L1, R11 to R4, R12 to R5, R13 to R6, U7 to U3

Commit message: Fixed diode layout, added C to VBUS and protection to BUCK-LDO interface
Changed lines of the file:
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@@
 		)
 		(fill
-			(type none)
+			(type color)
+			(color 92 0 255 0.168627451)
 		)
 		(effects
@@
 	(wire
 		(pts
-			(xy 203.2 76.2) (xy 223.52 76.2)
+			(xy 203.2 76.2) (xy 254 76.2)
 		)
 		(stroke
@@
 	(hierarchical_label "output_at_5.3"
 		(shape output)
-		(at 223.52 76.2 0)
+		(at 254 76.2 0)
 		(effects
 			(font
