File: POWERBOARD v3/power_v3.1/Conversion battery-5.3V_v3.1.kicad_sch (KiCad schematic)
At the start: 14 parts, among them U3 TPS62160DSG

Commit message: Added a comparator circuit that disables the buck converter when temp is too high and re enables it when it reaches a lower temperature
Connections:
- net at BUCK1IN1.2 (Pin_2), Cin1.1, U3.2 (VIN): no longer U3.3 (EN)
- new net EN: U3.3 (EN)
Changed lines of the file:
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@@
-	)
-	(junction
-		(at 119.38 97.79)
-		(diameter 0)
-		(color 0 0 0 0)
 	)
 	(junction
@@
 	(wire
 		(pts
-			(xy 119.38 95.25) (xy 119.38 97.79)
-		)
-		(stroke
-			(width 0)
-			(type default)
-		)
-	)
-	(wire
-		(pts
 			(xy 196.85 86.36) (xy 203.2 86.36)
 		)
@@
 	(wire
 		(pts
+			(xy 133.35 97.79) (xy 137.16 97.79)
+		)
+		(stroke
+			(width 0)
+			(type default)
+		)
+	)
+	(wire
+		(pts
 			(xy 149.86 113.03) (xy 149.86 119.38)
 		)
@@
 	(wire
 		(pts
-			(xy 119.38 97.79) (xy 137.16 97.79)
-		)
-		(stroke
-			(width 0)
-			(type default)
-		)
-	)
-	(wire
-		(pts
 			(xy 52.07 92.71) (xy 52.07 85.09)
 		)
@@
 	(wire
 		(pts
-			(xy 119.38 97.79) (xy 119.38 102.87)
+			(xy 119.38 95.25) (xy 119.38 102.87)
 		)
 		(stroke
@@
 		)
 	)
+	(global_label "EN"
+		(shape input)
+		(at 133.35 97.79 180)
+		(fields_autoplaced yes)
+		(effects
+			(font
+				(size 1.27 1.27)
+			)
+			(justify right)
+		)
+		(property "Intersheetrefs" "${INTERSHEET_REFS}"
+			(at 127.8853 97.79 0)
+			(hide yes)
+			(show_name no)
+			(do_not_autoplace no)
+			(effects
+				(font
+					(size 1.27 1.27)
+				)
+				(justify right)
+			)
+		)
+	)
