File: POWERBOARD v3/power_v3.1/power_v3.1.kicad_sch (KiCad schematic)
At the start: 0 parts

Commit message: Final changes before v3.2
Other:
- sheet 5.3V to 5V ports: added input_at_5.3; removed none
- sheet Recharge ports: added SYS; removed none
- sheet battery - 5.3V ports: added SYS, output_at_5.3; removed none
Changed lines of the file:
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@@
+			)
+		)
+		(pin "SYS" output
+			(at 102.87 107.95 0)
+			(effects
+				(font
+					(size 1.27 1.27)
+				)
+				(justify right)
 			)
 		)
@@
 			)
 		)
+		(pin "output_at_5.3" output
+			(at 153.67 107.95 0)
+			(effects
+				(font
+					(size 1.27 1.27)
+				)
+				(justify right)
+			)
+		)
+		(pin "SYS" input
+			(at 124.46 107.95 180)
+			(effects
+				(font
+					(size 1.27 1.27)
+				)
+				(justify left)
+			)
+		)
 		(instances
 			(project "power_v3.1"
@@
 			)
 		)
+		(pin "input_at_5.3" input
+			(at 175.26 107.95 180)
+			(effects
+				(font
+					(size 1.27 1.27)
+				)
+				(justify left)
+			)
+		)
