File: POWERBOARD v3/power_v3.2/RECHARGE_v3.2.kicad_sch (KiCad schematic)
At the start: 30 parts, among them J1 B2B_PH_K_S, J2 USB_C_Receptacle_USB2.0_16P, J4 R14 - 103AT-2, U1 TPS709-Q1, U2 USBLC6-2, U4 BQ25886RGE

Commit message: added TMP300 IC to measure temperature and corresponding resistor values
Parts:
- removed C5: 2.2u, symbol Device:C
- removed U1: TPS709-Q1, TPS70933DBVR:SOT95P280X145-5N, symbol Custom:TPS70933DBVR
- added R4: 316k, symbol Device:R
- added R5: 10k, symbol Device:R
- added U1: TMP300-Q1, symbol Customv3.2:TMP300-Q1
- C1: value 1u -> 0.1u
Connections:
- net EN: now also R5.1, U1.3 (OUT)
- net GND: now also R4.2, U1.2 (GND), U1.4 (HYSTSET)
- net SYS: now also C1.1, R5.2, U1.6 (V+)
- net BAT: no longer names the net of C11.1, CHAR/BATT1.1 (Pin_1), U4.13 (BAT), U4.14 (BAT)
- net BAT: no longer C1.1
- new net: R4.1, U1.1 (TSET)
