File: POWERBOARD v3/power_v3.3/5.3to5V_v3.3.kicad_sch (KiCad schematic)
At the start: 8 parts, among them IC1 MAX25301AATB_V+T

Commit message: added footprints
Parts:
- removed 5V1: TestPoint, TestPoint:TestPoint_Keystone_5000-5004_Miniature, symbol Connector:TestPoint
- removed 5V2: Conn_01x02, Connector_PinHeader_2.00mm:PinHeader_1x02_P2.00mm_Vertical, symbol Connector_Generic:Conn_01x02
- added J3: 2053380002, footprintsmolex:CONN_2053380000-SD_02_MOL, symbol 2026-10-07_20-29-31:2053380002
- added LDO5V1: TestPoint, TestPoint:TestPoint_Keystone_5000-5004_Miniature, symbol Connector:TestPoint
- C10, C12: footprint (none) -> Capacitor_SMD:C_0805_2012Metric
- C11: footprint (none) -> Capacitor_SMD:C_0402_1005Metric
- D3: footprint Diode_THT:D_DO-41_SOD81_P10.16mm_Horizontal -> Package_TO_SOT_SMD:SOT-23
- D4: footprint Diode_THT:D_DO-41_SOD81_P10.16mm_Horizontal -> Diode_SMD:D_SOD-128
Connections:
- net GND: now also J3.2
- net output_at_5: now also J3.1, LDO5V1.1
Changed lines of the file:
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@@
 			)
 		)
-		(property "Footprint" ""
+		(property "Footprint" "Capacitor_SMD:C_0805_2012Metric"
 			(at 101.2952 129.54 0)
 			(hide yes)
@@
 			)
 		)
-		(property "Footprint" ""
+		(property "Footprint" "Capacitor_SMD:C_0805_2012Metric"
 			(at 196.5452 90.17 0)
 			(hide yes)
@@
 	)
 	(symbol
+		(lib_id "Connector:TestPoint")
+		(at 207.01 67.31 0)
+		(unit 1)
+		(body_style 1)
+		(exclude_from_sim no)
+		(in_bom yes)
+		(on_board yes)
+		(in_pos_files yes)
+		(dnp no)
+		(fields_autoplaced yes)
+		(property "Reference" "LDO5V1"
+			(at 209.55 62.7379 0)
+			(show_name no)
+			(do_not_autoplace no)
+			(effects
+				(font
+					(size 1.27 1.27)
+				)
+				(justify left)
+			)
+		)
+		(property "Value" "TestPoint"
+			(at 209.55 65.2779 0)
+			(show_name no)
+			(do_not_autoplace no)
+			(effects
+				(font
+					(size 1.27 1.27)
+				)
+				(justify left)
+			)
+		)
+		(property "Footprint" "TestPoint:TestPoint_Keystone_5000-5004_Miniature"
+			(at 212.09 67.31 0)
+			(hide yes)
+			(show_name no)
+			(do_not_autoplace no)
+			(effects
+				(font
+					(size 1.27 1.27)
+				)
+			)
+		)
+		(property "Datasheet" ""
+			(at 212.09 67.31 0)
+			(hide yes)
+			(show_name no)
+			(do_not_autoplace no)
+			(effects
+				(font
+					(size 1.27 1.27)
+				)
+			)
+		)
+		(property "Description" "test point"
+			(at 207.01 67.31 0)
+			(hide yes)
+			(show_name no)
+			(do_not_autoplace no)
+			(effects
+				(font
+					(size 1.27 1.27)
+				)
+			)
+		)
+		(pin "1"
+		)
+		(instances
+			(project "power_v3.3"
+				(path "/432bcdcf-747a-4fa0-b87b-096f44260199/9585df76-13b3-4fa5-b448-53940051778a"
+					(reference "LDO5V1")
+					(unit 1)
+				)
+			)
+		)
+	)
+	(symbol
+		(lib_id "2026-10-07_20-29-31:2053380002")
+		(at 215.9 80.01 0)
+		(unit 1)
+		(body_style 1)
+		(exclude_from_sim no)
+		(in_bom yes)
+		(on_board yes)
+		(in_pos_files yes)
+		(dnp no)
+		(fields_autoplaced yes)
+		(property "Reference" "J3"
+			(at 229.87 80.0099 0)
+			(show_name no)
+			(do_not_autoplace no)
+			(effects
+				(font
+					(size 1.524 1.524)
+				)
+				(justify left)
+			)
+		)
+		(property "Value" "2053380002"
+			(at 229.87 82.5499 0)
+			(show_name no)
+			(do_not_autoplace no)
+			(effects
+				(font
+					(size 1.524 1.524)
+				)
+				(justify left)
+			)
+		)
+		(property "Footprint" "footprintsmolex:CONN_2053380000-SD_02_MOL"
+			(at 215.9 80.01 0)
+			(hide yes)
+			(show_name no)
+			(do_not_autoplace no)
+			(effects
+				(font
+					(size 1.27 1.27)
+					(italic yes)
+				)
+			)
+		)
+		(property "Datasheet" "https://www.molex.com/en-us/products/part-detail-pdf/2053380002?display=pdf"
+			(at 215.9 80.01 0)
+			(hide yes)
+			(show_name no)
+			(do_not_autoplace no)
+			(effects
+				(font
+					(size 1.27 1.27)
+					(italic yes)
+				)
+			)
+		)
+		(property "Description" ""
+			(at 215.9 80.01 0)
+			(hide yes)
+			(show_name no)
+			(do_not_autoplace no)
+			(effects
+				(font
+					(size 1.27 1.27)
+				)
+			)
+		)
+		(pin "2"
+		)
+		(pin "1"
+		)
+		(instances
+			(project "power_v3.3"
+				(path "/432bcdcf-747a-4fa0-b87b-096f44260199/9585df76-13b3-4fa5-b448-53940051778a"
+					(reference "J3")
+					(unit 1)
+				)
+			)
+		)
+	)
+	(symbol
 		(lib_id "Device:D_Zener")
 		(at 91.44 85.09 270)
@@
 			)
 		)
-		(property "Footprint" "Diode_THT:D_DO-41_SOD81_P10.16mm_Horizontal"
+		(property "Footprint" "Package_TO_SOT_SMD:SOT-23"
 			(at 91.44 85.09 0)
 			(hide yes)
@@
 			)
 		)
-		(property "Footprint" ""
+		(property "Footprint" "Capacitor_SMD:C_0402_1005Metric"
 			(at 116.5352 129.54 0)
 			(hide yes)
@@
 	)
 	(symbol
-		(lib_id "Connector_Generic:Conn_01x02")
-		(at 220.98 80.01 0)
-		(unit 1)
-		(body_style 1)
-		(exclude_from_sim no)
-		(in_bom yes)
-		(on_board yes)
-		(in_pos_files yes)
-		(dnp no)
-		(fields_autoplaced yes)
-		(property "Reference" "5V2"
-			(at 223.52 80.0099 0)
-			(show_name no)
-			(do_not_autoplace no)
-			(effects
-				(font
-					(size 1.27 1.27)
-				)
-				(justify left)
-			)
-		)
-		(property "Value" "Conn_01x02"
-			(at 223.52 82.5499 0)
-			(show_name no)
-			(do_not_autoplace no)
-			(effects
-				(font
-					(size 1.27 1.27)
-				)
-				(justify left)
-			)
-		)
-		(property "Footprint" "Connector_PinHeader_2.00mm:PinHeader_1x02_P2.00mm_Vertical"
-			(at 220.98 80.01 0)
-			(hide yes)
-			(show_name no)
-			(do_not_autoplace no)
-			(effects
-				(font
-					(size 1.27 1.27)
-				)
-			)
-		)
-		(property "Datasheet" ""
-			(at 220.98 80.01 0)
-			(hide yes)
-			(show_name no)
-			(do_not_autoplace no)
-			(effects
-				(font
-					(size 1.27 1.27)
-				)
-			)
-		)
-		(property "Description" "Generic connector, single row, 01x02, script generated (kicad-library-utils/schlib/autogen/connector/)"
-			(at 220.98 80.01 0)
-			(hide yes)
-			(show_name no)
-			(do_not_autoplace no)
-			(effects
-				(font
-					(size 1.27 1.27)
-				)
-			)
-		)
-		(pin "2"
-		)
-		(pin "1"
-		)
-		(instances
-			(project "power_v3.3"
-				(path "/432bcdcf-747a-4fa0-b87b-096f44260199/9585df76-13b3-4fa5-b448-53940051778a"
-					(reference "5V2")
-					(unit 1)
-				)
-			)
-		)
-	)
-	(symbol
-		(lib_id "Connector:TestPoint")
-		(at 207.01 67.31 0)
-		(unit 1)
-		(body_style 1)
-		(exclude_from_sim no)
-		(in_bom yes)
-		(on_board yes)
-		(in_pos_files yes)
-		(dnp no)
-		(property "Reference" "5V1"
-			(at 207.264 57.658 0)
-			(show_name no)
-			(do_not_autoplace no)
-			(effects
-				(font
-					(size 1.27 1.27)
-				)
-				(justify left)
-			)
-		)
-		(property "Value" "TestPoint"
-			(at 207.772 61.468 0)
-			(show_name no)
-			(do_not_autoplace no)
-			(effects
-				(font
-					(size 1.27 1.27)
-				)
-				(justify left)
-			)
-		)
-		(property "Footprint" "TestPoint:TestPoint_Keystone_5000-5004_Miniature"
-			(at 212.09 67.31 0)
-			(hide yes)
-			(show_name no)
-			(do_not_autoplace no)
-			(effects
-				(font
-					(size 1.27 1.27)
-				)
-			)
-		)
-		(property "Datasheet" ""
-			(at 212.09 67.31 0)
-			(hide yes)
-			(show_name no)
-			(do_not_autoplace no)
-			(effects
-				(font
-					(size 1.27 1.27)
-				)
-			)
-		)
-		(property "Description" "test point"
-			(at 207.01 67.31 0)
-			(hide yes)
-			(show_name no)
-			(do_not_autoplace no)
-			(effects
-				(font
-					(size 1.27 1.27)
-				)
-			)
-		)
-		(pin "1"
-		)
-		(instances
-			(project "power_v3.3"
-				(path "/432bcdcf-747a-4fa0-b87b-096f44260199/9585df76-13b3-4fa5-b448-53940051778a"
-					(reference "5V1")
-					(unit 1)
-				)
-			)
-		)
-	)
-	(symbol
 		(lib_id "Device:D_Zener")
 		(at 170.18 86.36 270)
@@
 			)
 		)
-		(property "Footprint" "Diode_THT:D_DO-41_SOD81_P10.16mm_Horizontal"
+		(property "Footprint" "Diode_SMD:D_SOD-128"
 			(at 170.18 86.36 0)
 			(hide yes)

Commit message: finished footprint assignment, added on-off general switch
Parts:
- IC1: footprint N_pulse:SON50P300X300X80-11N -> MAX25301AATB_V+T:SON50P300X300X80-11N
Other:
- note added: "ajouter buzzer + système de switch des machins"
Changed lines of the file:
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@@
+		)
+	)
+	(text "ajouter buzzer + système de switch des machins"
+		(exclude_from_sim no)
+		(at 63.754 31.496 0)
+		(effects
+			(font
+				(size 1.27 1.27)
+			)
 		)
 	)
@@
 			)
 		)
-		(property "Footprint" "N_pulse:SON50P300X300X80-11N"
+		(property "Footprint" "MAX25301AATB_V+T:SON50P300X300X80-11N"
 			(at 151.13 168.58 0)
 			(hide yes)

Commit message: (nearly) finished schematic and layout, beginning routing (hooooooly)
Parts:
- added C14, C15, C16, C17: 100n, Capacitor_SMD:C_0402_1005Metric, symbol Device:C
- added D5: LED, LED_THT:LED_D5.0mm, symbol Device:LED
- added IC2: MCP6541T-I_OT, MCP6541T-I_OT:SOT95P270X145-5N, symbol MCP6541T-I_OT:MCP6541T-I_OT
- added IC3: AP2281-1FMG-7, APP2281-1FMG-7:SON50P201X181X60-7N, symbol AP2281-1FMG-7:AP2281-1FMG-7
- added R13, R15, R17: 10k, Resistor_SMD:R_0603_1608Metric, symbol Device:R
- added R14: 51.1k, Resistor_SMD:R_0603_1608Metric, symbol Device:R
- added R16: 26.7k, Resistor_SMD:R_0603_1608Metric, symbol Device:R
- added R18: 330, Resistor_SMD:R_0603_1608Metric, symbol Device:R
- added S2: MFS201N-9-Z, MFS201N-9-Z:MFS201N9Z, symbol MFS201N-9-Z:MFS201N-9-Z
- renumbered LDO5V1 to LDO5V
Connections:
- net GND: now also C14.2, C15.2, C16.2, C17.2, IC2.2 (VSS), IC3.4 (GND_1), IC3.7 (GND_2), R13.1, R17.2
- net output_at_5: now also C15.1, D5.2 (A), IC2.5 (VDD), IC3.1 (IN_1), IC3.2 (IN_2), R15.1, R16.1; no longer J3.1
- new net: C14.1, IC2.4 (VIN-), R16.2, R17.1
- new net: C17.1, IC3.5 (OUT_1), IC3.6 (OUT_2), J3.1
- new net: D5.1 (K), R18.1
- new net: S2.1 (NO_1), S2.4 (NO_2)
- new net: R13.2, S2.6 (NC_2)
- new net INCOMP: C16.1, IC2.3 (VIN+), R14.2, R15.2, S2.3 (NC_1)
- new net NTC: S2.2 (COM_1)
- new net TS: S2.5 (COM_2)
- new net switch_out: IC2.1 (OUT), IC3.3 (EN), R14.1, R18.2
- no-connect marks 0 -> 2
Other:
- note removed: "ajouter buzzer + système de switch des machins"
- moved on the sheet: C10, C11, C12, D3, D4, IC1, J3, LDO5V

Commit message: updated routing
Parts:
- renumbered LDO5V to LDO5V1
Changed lines of the file:
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@@
 		(dnp no)
 		(fields_autoplaced yes)
-		(property "Reference" "LDO5V"
+		(property "Reference" "LDO5V1"
 			(at 208.28 46.2279 0)
 			(show_name no)
@@
 			(project "power_v3.3"
 				(path "/432bcdcf-747a-4fa0-b87b-096f44260199/9585df76-13b3-4fa5-b448-53940051778a"
-					(reference "LDO5V")
+					(reference "LDO5V1")
 					(unit 1)
 				)
